Commit message: added new endeffector and Table

File: iiwa_nadelhalterung/iiwa_nadelhalterung_description/urdf/iiwa_nadelhalterung.urdf.xacro (robot description, xacro)
@@ -15,29 +15,104 @@
   -->
   <!--     <link name="world"/> -->
-  <link name="world">
+<material name="wood">
+    <color rgba="0.89 0.58 0.47 0.3"/>
+  </material>
+  <material name="aluminium">
+    <color rgba="0.7 0.7 0.7 0.4"/>
+  </material>
+  <link name="world"/>
+  <joint name="world_table" type="fixed">
+    <parent link="world" />
+    <child link="table" />
+  </joint>
+  <!-- Create table on which iiwa is standing -->
+  <link name="table">
+    <inertial>
+      <origin xyz="0.0 0.0 0.5" rpy="0 0 0"/>
+      <mass value="15"/>
+      <inertia ixx="0.05"  ixy="0"  ixz="0" iyy="0.06" iyz="0" izz="0.03" />
+    </inertial>
     <visual>
-      <origin xyz="0 0 0.42" rpy="0 0 0"/>
+      <origin xyz="0 0 0.70" rpy="0 0 0"/>
       <geometry>
-	<box size="0.68 0.605 0.84"/>
+        <box size="1.5 1.5 0.04"/>
       </geometry>
+      <material name="wood"/>
+    </visual>
+    <visual>
+      <origin xyz="0.66 0.66 0.34" rpy="0 0 0"/>
+      <geometry>
+        <box size="0.08 0.08 0.68"/>
+      </geometry>
+      <material name="aluminium"/>
+    </visual>
+    <visual>
+      <origin xyz="-0.66 0.66 0.34" rpy="0 0 0"/>
+      <geometry>
+        <box size="0.08 0.08 0.68"/>
+      </geometry>
+      <material name="aluminium"/>
+    </visual>
+    <visual>
+      <origin xyz="0.66 -0.66 0.34" rpy="0 0 0"/>
+      <geometry>
+        <box size="0.08 0.08 0.68"/>
+      </geometry>
+      <material name="aluminium"/>
+    </visual>
+    <visual>
+      <origin xyz="-0.66 -0.66 0.34" rpy="0 0 0"/>
+      <geometry>
+        <box size="0.08 0.08 0.68"/>
+      </geometry>
+      <material name="aluminium"/>
     </visual>
     <collision>
-      <origin xyz="0 0 0.42" rpy="0 0 0"/>
+      <origin xyz="0 0 0.70" rpy="0 0 0"/>
       <geometry>
-	<box size="0.68 0.605 0.84"/>
+        <box size="1.5 1.5 0.04"/>
       </geometry>
+      <material name="wood"/>
+    </collision>
+    <collision>
+      <origin xyz="0.66 0.66 0.34" rpy="0 0 0"/>
+      <geometry>
+        <box size="0.08 0.08 0.68"/>
+      </geometry>
+      <material name="aluminium"/>
+    </collision>
+    <collision>
+      <origin xyz="-0.66 0.66 0.34" rpy="0 0 0"/>
+      <geometry>
+        <box size="0.08 0.08 0.68"/>
+      </geometry>
+      <material name="aluminium"/>
+    </collision>
+    <collision>
+      <origin xyz="0.66 -0.66 0.34" rpy="0 0 0"/>
+      <geometry>
+        <box size="0.08 0.08 0.68"/>
+      </geometry>
+      <material name="aluminium"/>
+    </collision>
+    <collision>
+      <origin xyz="-0.66 -0.66 0.34" rpy="0 0 0"/>
+      <geometry>
+        <box size="0.08 0.08 0.68"/>
+      </geometry>
+      <material name="aluminium"/>
     </collision>
   </link>
-  <gazebo reference="world">
+  <gazebo reference="table">
     <static>true</static>
   </gazebo>
   <!-- Here we insert an iiwa14 robot in the scene, it's origin is just on top of the box previously defined. You can use 0,0,0 if you don't have that. -->
-  <xacro:iiwa14 hardware_interface="$(arg hardware_interface)" robot_name="$(arg robot_name)" parent="world">
-    <origin xyz="0 0 0.84" rpy="0 0 0"/>
+  <xacro:iiwa14 hardware_interface="$(arg hardware_interface)" robot_name="$(arg robot_name)" parent="table">
+    <origin xyz="0 0 0.72" rpy="0 0 0"/>
   </xacro:iiwa14>
   <!-- Tool properties -->
-  <property name="tool_mass" value="0.0200" />
-  <property name="tool_joint_offset" value="0.00 0.00 0.00" />
-  <property name="tool_link_offset" value="-0.015 0.0075 0.058" />
+  <xacro:property name="tool_mass" value="0.0200" />
+  <xacro:property name="tool_joint_offset" value="0.0275 0.00 0.00" />
+  <xacro:property name="tool_link_offset" value="-0.015 0.0075 0.058" />
   <!--  Here we define a dummy joint between the tip of the iiwa14 and the base of the tool.
   There is no offset between the two, that means the tool is attached at the robot flange. -->
@@ -45,5 +120,5 @@
     <parent link="iiwa_link_ee" />
     <child link = "tool_link" />
-    <origin xyz="${tool_joint_offset}" rpy="0 0 0" />
+     <origin xyz="${tool_joint_offset}" rpy="0 0 0" />
   </joint>
   <!-- Here we define the geometry of the tool. We designed the tool ourselves, so we have a mesh file that represents it.
@@ -51,7 +126,7 @@
   <link name="tool_link">
     <visual>
-      <origin xyz="0 0 0" rpy="0 0 0"/>
+      <origin xyz="${tool_joint_offset}" rpy="0 0 ${3*PI/2.0}"/>
       <geometry>
-	<mesh filename="package://iiwa_nadelhalterung_description/meshes/visual/EEF_plusFlansch.stl" />
+	<mesh filename="package://iiwa_nadelhalterung_description/meshes/visual/eef.stl" />
 	<!-- 	<cylinder length="0.1275" radius="0.020"/> -->
       </geometry>
@@ -59,7 +134,7 @@
     </visual>
     <collision>
-      <origin xyz="0 0 0" rpy="0 0 0"/>
+      <origin xyz="${tool_joint_offset}" rpy="0 0 ${PI/2.0}"/>
       <geometry>
-	<mesh filename="package://iiwa_nadelhalterung_description/meshes/visual/EEF_plusFlansch.stl" />
+	<mesh filename="package://iiwa_nadelhalterung_description/meshes/visual/eef.stl" />
 	<!-- 	<cylinder length="0.1275" radius="0.020"/> -->
       </geometry>

Commit message: changed .setupAssistant setting

File: iiwa_nadelhalterung/iiwa_nadelhalterung_description/urdf/iiwa_nadelhalterung.urdf.xacro (robot description, xacro)
@@ -114,5 +114,5 @@
   <xacro:property name="tool_mass" value="0.0200" />
   <xacro:property name="tool_joint_offset" value="0.0275 0.00 0.00" />
-  <xacro:property name="tool_link_offset" value="-0.015 0.0075 0.058" />
+  <xacro:property name="tool_link_offset" value="0.085 0.0075 0.079" />
   <!--  Here we define a dummy joint between the tip of the iiwa14 and the base of the tool.
   There is no offset between the two, that means the tool is attached at the robot flange. -->

Commit message: some changes

File: iiwa_nadelhalterung/iiwa_nadelhalterung_description/urdf/iiwa_nadelhalterung.urdf.xacro (robot description, xacro)
@@ -14,5 +14,4 @@
   If you don't want to have that you can define a basic world link (see commented lines)
   -->
-  <!--     <link name="world"/> -->
 <material name="wood">
     <color rgba="0.89 0.58 0.47 0.3"/>
@@ -147,5 +146,5 @@
     <parent link="tool_link" />
     <child link = "tool_link_ee" />
-    <origin xyz="${tool_link_offset}" rpy="0 0 0" />
+    <origin xyz="${tool_link_offset}" rpy="0 ${-PI/2} ${PI/2}" />
   </joint>
   <!--  The TCP frame is here defined -->

Commit message: configured new eef

File: iiwa_nadelhalterung/iiwa_nadelhalterung_description/urdf/iiwa_nadelhalterung.urdf.xacro (robot description, xacro)
@@ -112,6 +112,7 @@
   <!-- Tool properties -->
   <xacro:property name="tool_mass" value="0.0200" />
-  <xacro:property name="tool_joint_offset" value="0.0275 0.00 0.00" />
-  <xacro:property name="tool_link_offset" value="0.085 0.0075 0.079" />
+  <xacro:property name="tool_joint_offset" value="0.0275 0.00 0.00" /> <!-- to get the .stl file in place -> does NOT define the toolframe-->
+  <xacro:property name="tool_link_ee_offset" value="0.1125 -0.0075 0.0795" />
+  <xacro:property name="tool_link_nh_offset" value="0.0 -0.0075 -0.0075" /> <!-- relative to tool_link_ee -> get values from file! -->
   <!--  Here we define a dummy joint between the tip of the iiwa14 and the base of the tool.
   There is no offset between the two, that means the tool is attached at the robot flange. -->
@@ -142,11 +143,17 @@
   </link>
   <!--  Here we define another dummy joint. It is placed at the end of the tool, so we can then attach a frame at its TCP for control -->
-  <!-- For registration the dummy joint coincides with the corner of the registration-tool-part of nadelhalterung -> x= -->
-   <joint name="tool_tip_joint" type="fixed">
-    <parent link="tool_link" />
+  <!-- For registration the dummy joint coincides with the corner of the registration-part of the tool  -> x= -->
+   <joint name="tool_tip_ee_joint" type="fixed">
+    <parent link="iiwa_link_ee" />
     <child link = "tool_link_ee" />
-    <origin xyz="${tool_link_offset}" rpy="0 ${-PI/2} ${PI/2}" />
+    <origin xyz="${tool_link_ee_offset}" rpy="0 ${-PI/2} ${PI/2}" />
   </joint>
+  <!--<joint name="tool_tip_nh_joint" type="fixed">
+    <parent link="tool_link_ee" />
+    <child link = "tool_link_nh" />
+    <origin xyz="${tool_link_nh_offset}" rpy="0 0 0" />
+  </joint>-->
   <!--  The TCP frame is here defined -->
   <link name="tool_link_ee"/>
+  <!--link name="tool_link_nh"/--> <!--only if needed-->
 </robot>

Commit message: included toolbar.launch ro movie_planning_exe..

File: iiwa_nadelhalterung/iiwa_nadelhalterung_description/urdf/iiwa_nadelhalterung.urdf.xacro (robot description, xacro)
@@ -147,5 +147,5 @@
     <parent link="iiwa_link_ee" />
     <child link = "tool_link_ee" />
-    <origin xyz="${tool_link_ee_offset}" rpy="0 ${-PI/2} ${PI/2}" />
+    <origin xyz="${tool_link_ee_offset}" rpy="${-PI/2} ${-PI/2} 0" />
   </joint>
   <!--<joint name="tool_tip_nh_joint" type="fixed">
